Commit message: Removed walls from complex_env.urdf, moved the mesh directory for dual_arm.urdf

File: data/urdfs/complex_env/complex_env.urdf (robot description, URDF)
Before this commit: robot dual_arm, 9 links, 8 joints
Links:
- removed link floor
- removed link left_arm_base
- removed link plexiglass
- removed link right_arm_base
- removed link table
- removed link table_at_front
- removed link window
- removed link windowsill
Joints:
- removed joint floor_joint
- removed joint plexiglass_joint
- removed joint table_at_front_joint
- removed joint table_joint
- removed joint ur10_base_joint_connection
- removed joint ur5_base_joint_connection
- removed joint window_joint
- removed joint windowsill_joint

File: data/urdfs/dual_arm/dual_arm.urdf (robot description, URDF)
Before this commit: robot dual_arm, 25 links, 24 joints
Links:
- link ur10_base_link_inertia: geometry collision mesh filename=meshes/ur10/collision/base.stl; visual mesh filename=meshes/ur10/visual/base.obj
- link ur10_forearm_link: geometry collision mesh filename=meshes/ur10/collision/forearm.stl; visual mesh filename=meshes/ur10/visual/forearm.obj
- link ur10_shoulder_link: geometry collision mesh filename=meshes/ur10/collision/shoulder.stl; visual mesh filename=meshes/ur10/visual/shoulder.obj
- link ur10_upper_arm_link: geometry collision mesh filename=meshes/ur10/collision/upperarm.stl; visual mesh filename=meshes/ur10/visual/upperarm.obj
- link ur10_wrist_1_link: geometry collision mesh filename=meshes/ur10/collision/wrist1.stl; visual mesh filename=meshes/ur10/visual/wrist1.obj
- link ur10_wrist_2_link: geometry collision mesh filename=meshes/ur10/collision/wrist2.stl; visual mesh filename=meshes/ur10/visual/wrist2.obj
- link ur10_wrist_3_link: geometry collision mesh filename=meshes/ur10/collision/wrist3.stl; visual mesh filename=meshes/ur10/visual/wrist3.obj
- link ur5_base_link_inertia: geometry collision mesh filename=meshes/ur5/collision/base.stl; visual mesh filename=meshes/ur5/visual/base.obj
- link ur5_forearm_link: geometry collision mesh filename=meshes/ur5/collision/forearm.stl; visual mesh filename=meshes/ur5/visual/forearm.obj
- link ur5_shoulder_link: geometry collision mesh filename=meshes/ur5/collision/shoulder.stl; visual mesh filename=meshes/ur5/visual/shoulder.obj
- link ur5_upper_arm_link: geometry collision mesh filename=meshes/ur5/collision/upperarm.stl; visual mesh filename=meshes/ur5/visual/upperarm.obj
- link ur5_wrist_1_link: geometry collision mesh filename=meshes/ur5/collision/wrist1.stl; visual mesh filename=meshes/ur5/visual/wrist1.obj
- link ur5_wrist_2_link: geometry collision mesh filename=meshes/ur5/collision/wrist2.stl; visual mesh filename=meshes/ur5/visual/wrist2.obj
- link ur5_wrist_3_link: geometry collision mesh filename=meshes/ur5/collision/wrist3.stl; visual mesh filename=meshes/ur5/visual/wrist3.obj

Commit message: Added first version of the real complex environment

File: data/urdfs/complex_env/complex_env.urdf (robot description, URDF)
Before this commit: robot dual_arm_env, 1 links, 0 joints
Links:
- added link a_toy_airplane_12; collision mesh filename=meshes/ycb-google_64k/a_toy_airplane/nontextured.stl; visual mesh filename=meshes/ycb-google_64k/a_toy_airplane/nontextured.stl
- added link a_toy_airplane_16; collision mesh filename=meshes/ycb-google_64k/a_toy_airplane/nontextured.stl; visual mesh filename=meshes/ycb-google_64k/a_toy_airplane/nontextured.stl
- added link banana_10; collision mesh filename=meshes/ycb-google_64k/banana/nontextured.stl; visual mesh filename=meshes/ycb-google_64k/banana/nontextured.stl
- added link banana_2; collision mesh filename=meshes/ycb-google_64k/banana/nontextured.stl; visual mesh filename=meshes/ycb-google_64k/banana/nontextured.stl
- added link banana_4; collision mesh filename=meshes/ycb-google_64k/banana/nontextured.stl; visual mesh filename=meshes/ycb-google_64k/banana/nontextured.stl
- added link bleach_cleanser_0; collision mesh filename=meshes/ycb-google_64k/bleach_cleanser/nontextured.stl; visual mesh filename=meshes/ycb-google_64k/bleach_cleanser/nontextured.stl
- added link bowl_19; collision mesh filename=meshes/ycb-google_64k/bowl/nontextured.stl; visual mesh filename=meshes/ycb-google_64k/bowl/nontextured.stl
- added link bowl_9; collision mesh filename=meshes/ycb-google_64k/bowl/nontextured.stl; visual mesh filename=meshes/ycb-google_64k/bowl/nontextured.stl
- added link cracker_box_18; collision mesh filename=meshes/ycb-google_64k/cracker_box/nontextured.stl; visual mesh filename=meshes/ycb-google_64k/cracker_box/nontextured.stl
- added link cracker_box_3; collision mesh filename=meshes/ycb-google_64k/cracker_box/nontextured.stl; visual mesh filename=meshes/ycb-google_64k/cracker_box/nontextured.stl
- added link left_arm_base
- added link mug_13; collision mesh filename=meshes/ycb-google_64k/mug/nontextured.stl; visual mesh filename=meshes/ycb-google_64k/mug/nontextured.stl
- added link mug_14; collision mesh filename=meshes/ycb-google_64k/mug/nontextured.stl; visual mesh filename=meshes/ycb-google_64k/mug/nontextured.stl
- added link mug_8; collision mesh filename=meshes/ycb-google_64k/mug/nontextured.stl; visual mesh filename=meshes/ycb-google_64k/mug/nontextured.stl
- added link powerdrill_11; collision mesh filename=meshes/ycb-google_64k/powerdrill/nontextured.stl; visual mesh filename=meshes/ycb-google_64k/powerdrill/nontextured.stl
- added link powerdrill_17; collision mesh filename=meshes/ycb-google_64k/powerdrill/nontextured.stl; visual mesh filename=meshes/ycb-google_64k/powerdrill/nontextured.stl
- added link powerdrill_5; collision mesh filename=meshes/ycb-google_64k/powerdrill/nontextured.stl; visual mesh filename=meshes/ycb-google_64k/powerdrill/nontextured.stl
- added link powerdrill_6; collision mesh filename=meshes/ycb-google_64k/powerdrill/nontextured.stl; visual mesh filename=meshes/ycb-google_64k/powerdrill/nontextured.stl
- added link powerdrill_7; collision mesh filename=meshes/ycb-google_64k/powerdrill/nontextured.stl; visual mesh filename=meshes/ycb-google_64k/powerdrill/nontextured.stl
- added link right_arm_base
- added link strawberry_1; collision mesh filename=meshes/ycb-google_64k/strawberry/nontextured.stl; visual mesh filename=meshes/ycb-google_64k/strawberry/nontextured.stl
- added link strawberry_15; collision mesh filename=meshes/ycb-google_64k/strawberry/nontextured.stl; visual mesh filename=meshes/ycb-google_64k/strawberry/nontextured.stl
Joints:
- added joint a_toy_airplane_12_joint: type fixed, parent left_arm_base, child a_toy_airplane_12, origin xyz=-0.95625 0.57020 0.00176 rpy=0.25202 1.79978 -1.06099
- added joint a_toy_airplane_16_joint: type fixed, parent right_arm_base, child a_toy_airplane_16, origin xyz=-0.54569 -0.73351 0.28173 rpy=1.27313 -0.02203 -2.42411
- added joint banana_10_joint: type fixed, parent right_arm_base, child banana_10, origin xyz=0.12673 -0.15931 0.65268 rpy=2.75492 0.07854 -2.32949
- added joint banana_2_joint: type fixed, parent left_arm_base, child banana_2, origin xyz=0.09189 0.46243 0.24399 rpy=-1.32084 -3.00657 2.12106
- added joint banana_4_joint: type fixed, parent left_arm_base, child banana_4, origin xyz=0.67007 -0.42415 0.15334 rpy=-1.35617 2.97478 -0.00401
- added joint bleach_cleanser_0_joint: type fixed, parent right_arm_base, child bleach_cleanser_0, origin xyz=1.17892 0.22942 0.03057 rpy=0.26020 2.75926 -0.74642
- added joint bowl_19_joint: type fixed, parent right_arm_base, child bowl_19, origin xyz=-0.67386 -0.02673 0.31815 rpy=2.08756 2.99693 0.82166
- added joint bowl_9_joint: type fixed, parent left_arm_base, child bowl_9, origin xyz=-0.98236 -0.52246 0.57505 rpy=-1.44966 0.30157 2.87215
- added joint cracker_box_18_joint: type fixed, parent right_arm_base, child cracker_box_18, origin xyz=-0.25287 0.11580 1.23462 rpy=-1.72553 -0.64519 -2.91963
- added joint cracker_box_3_joint: type fixed, parent right_arm_base, child cracker_box_3, origin xyz=0.24773 -0.01161 0.41785 rpy=-2.38202 -1.05121 1.39163
- added joint mug_13_joint: type fixed, parent right_arm_base, child mug_13, origin xyz=-0.60808 -0.69298 0.60835 rpy=-2.00569 -2.56604 0.32063
- added joint mug_14_joint: type fixed, parent left_arm_base, child mug_14, origin xyz=0.31101 -0.11514 0.02342 rpy=2.31270 -0.29532 1.59684
- added joint mug_8_joint: type fixed, parent right_arm_base, child mug_8, origin xyz=0.50812 -0.05747 0.61814 rpy=0.24892 2.26377 -1.68279
- added joint powerdrill_11_joint: type fixed, parent right_arm_base, child powerdrill_11, origin xyz=0.33596 0.12364 0.63171 rpy=0.43982 -1.88596 0.02966
- added joint powerdrill_17_joint: type fixed, parent left_arm_base, child powerdrill_17, origin xyz=-0.59277 0.32144 0.12910 rpy=-2.45822 2.51213 0.06356
- added joint powerdrill_5_joint: type fixed, parent left_arm_base, child powerdrill_5, origin xyz=0.84220 0.18562 0.21580 rpy=1.86865 -0.53838 -2.05456
- added joint powerdrill_6_joint: type fixed, parent left_arm_base, child powerdrill_6, origin xyz=-0.19815 -0.32917 0.04171 rpy=-2.11305 2.13598 -0.81353
- added joint powerdrill_7_joint: type fixed, parent right_arm_base, child powerdrill_7, origin xyz=-0.14646 0.38013 0.65262 rpy=0.72138 0.49119 0.92461
- added joint strawberry_15_joint: type fixed, parent left_arm_base, child strawberry_15, origin xyz=0.33149 0.27245 0.34337 rpy=-0.97752 -2.70481 -2.13864
- added joint strawberry_1_joint: type fixed, parent right_arm_base, child strawberry_1, origin xyz=-0.16293 -1.06563 0.66958 rpy=1.65688 2.75937 0.33213
- added joint ur10_base_joint_connection: type fixed, parent world, child left_arm_base, origin xyz=0.9772262573242188 -0.026124268770217896 0.81 rpy=0.00000 0.00000 1.5708
- added joint ur5_base_joint_connection: type fixed, parent world, child right_arm_base, origin xyz=-0.4220163822174072 -0.10995670408010483 0.76 rpy=0.00000 0.00000 0.00000
