Commit message: Added hands to dual_arm.urdf, re-generated the benchmark cases

File: data/urdfs/complex_env/complex_env.urdf (robot description, URDF)
Before this commit: robot dual_arm_env, 23 links, 22 joints
Links:
- removed link a_toy_airplane_12
- removed link a_toy_airplane_16
- removed link banana_10
- removed link banana_4
- removed link bleach_cleanser_0
- removed link bowl_19
- removed link bowl_9
- removed link cracker_box_18
- removed link cracker_box_3
- removed link mug_8
- removed link powerdrill_11
- removed link powerdrill_17
- removed link powerdrill_5
- removed link powerdrill_6
- removed link powerdrill_7
- removed link strawberry_1
- removed link strawberry_15
- added link a_toy_airplane_0; collision mesh filename=meshes/ycb-google_64k/a_toy_airplane/nontextured.stl; visual mesh filename=meshes/ycb-google_64k/a_toy_airplane/nontextured.stl
- added link a_toy_airplane_10; collision mesh filename=meshes/ycb-google_64k/a_toy_airplane/nontextured.stl; visual mesh filename=meshes/ycb-google_64k/a_toy_airplane/nontextured.stl
- added link a_toy_airplane_21; collision mesh filename=meshes/ycb-google_64k/a_toy_airplane/nontextured.stl; visual mesh filename=meshes/ycb-google_64k/a_toy_airplane/nontextured.stl
- added link a_toy_airplane_22; collision mesh filename=meshes/ycb-google_64k/a_toy_airplane/nontextured.stl; visual mesh filename=meshes/ycb-google_64k/a_toy_airplane/nontextured.stl
- added link banana_1; collision mesh filename=meshes/ycb-google_64k/banana/nontextured.stl; visual mesh filename=meshes/ycb-google_64k/banana/nontextured.stl
- added link bleach_cleanser_12; collision mesh filename=meshes/ycb-google_64k/bleach_cleanser/nontextured.stl; visual mesh filename=meshes/ycb-google_64k/bleach_cleanser/nontextured.stl
- added link bleach_cleanser_29; collision mesh filename=meshes/ycb-google_64k/bleach_cleanser/nontextured.stl; visual mesh filename=meshes/ycb-google_64k/bleach_cleanser/nontextured.stl
- added link bleach_cleanser_4; collision mesh filename=meshes/ycb-google_64k/bleach_cleanser/nontextured.stl; visual mesh filename=meshes/ycb-google_64k/bleach_cleanser/nontextured.stl
- added link bowl_8; collision mesh filename=meshes/ycb-google_64k/bowl/nontextured.stl; visual mesh filename=meshes/ycb-google_64k/bowl/nontextured.stl
- added link cracker_box_20; collision mesh filename=meshes/ycb-google_64k/cracker_box/nontextured.stl; visual mesh filename=meshes/ycb-google_64k/cracker_box/nontextured.stl
- added link cracker_box_5; collision mesh filename=meshes/ycb-google_64k/cracker_box/nontextured.stl; visual mesh filename=meshes/ycb-google_64k/cracker_box/nontextured.stl
- added link cracker_box_6; collision mesh filename=meshes/ycb-google_64k/cracker_box/nontextured.stl; visual mesh filename=meshes/ycb-google_64k/cracker_box/nontextured.stl
- added link hammer_16; collision mesh filename=meshes/ycb-google_64k/hammer/nontextured.stl; visual mesh filename=meshes/ycb-google_64k/hammer/nontextured.stl
- added link hammer_23; collision mesh filename=meshes/ycb-google_64k/hammer/nontextured.stl; visual mesh filename=meshes/ycb-google_64k/hammer/nontextured.stl
- added link hammer_25; collision mesh filename=meshes/ycb-google_64k/hammer/nontextured.stl; visual mesh filename=meshes/ycb-google_64k/hammer/nontextured.stl
- added link hammer_3; collision mesh filename=meshes/ycb-google_64k/hammer/nontextured.stl; visual mesh filename=meshes/ycb-google_64k/hammer/nontextured.stl
- added link mug_26; collision mesh filename=meshes/ycb-google_64k/mug/nontextured.stl; visual mesh filename=meshes/ycb-google_64k/mug/nontextured.stl
- added link mug_27; collision mesh filename=meshes/ycb-google_64k/mug/nontextured.stl; visual mesh filename=meshes/ycb-google_64k/mug/nontextured.stl
- added link powerdrill_18; collision mesh filename=meshes/ycb-google_64k/powerdrill/nontextured.stl; visual mesh filename=meshes/ycb-google_64k/powerdrill/nontextured.stl
- added link powerdrill_24; collision mesh filename=meshes/ycb-google_64k/powerdrill/nontextured.stl; visual mesh filename=meshes/ycb-google_64k/powerdrill/nontextured.stl
- added link rubiks_cube_15; collision mesh filename=meshes/ycb-google_64k/rubiks_cube/nontextured.stl; visual mesh filename=meshes/ycb-google_64k/rubiks_cube/nontextured.stl
- added link rubiks_cube_17; collision mesh filename=meshes/ycb-google_64k/rubiks_cube/nontextured.stl; visual mesh filename=meshes/ycb-google_64k/rubiks_cube/nontextured.stl
- added link rubiks_cube_19; collision mesh filename=meshes/ycb-google_64k/rubiks_cube/nontextured.stl; visual mesh filename=meshes/ycb-google_64k/rubiks_cube/nontextured.stl
- added link rubiks_cube_28; collision mesh filename=meshes/ycb-google_64k/rubiks_cube/nontextured.stl; visual mesh filename=meshes/ycb-google_64k/rubiks_cube/nontextured.stl
- added link strawberry_11; collision mesh filename=meshes/ycb-google_64k/strawberry/nontextured.stl; visual mesh filename=meshes/ycb-google_64k/strawberry/nontextured.stl
- added link strawberry_7; collision mesh filename=meshes/ycb-google_64k/strawberry/nontextured.stl; visual mesh filename=meshes/ycb-google_64k/strawberry/nontextured.stl
- added link strawberry_9; collision mesh filename=meshes/ycb-google_64k/strawberry/nontextured.stl; visual mesh filename=meshes/ycb-google_64k/strawberry/nontextured.stl
Joints:
- removed joint a_toy_airplane_12_joint
- removed joint a_toy_airplane_16_joint
- removed joint banana_10_joint
- removed joint banana_4_joint
- removed joint bleach_cleanser_0_joint
- removed joint bowl_19_joint
- removed joint bowl_9_joint
- removed joint cracker_box_18_joint
- removed joint cracker_box_3_joint
- removed joint mug_8_joint
- removed joint powerdrill_11_joint
- removed joint powerdrill_17_joint
- removed joint powerdrill_5_joint
- removed joint powerdrill_6_joint
- removed joint powerdrill_7_joint
- removed joint strawberry_15_joint
- removed joint strawberry_1_joint
- added joint a_toy_airplane_0_joint: type fixed, parent right_arm_base, child a_toy_airplane_0, origin xyz=0.57273 0.08650 0.19915 rpy=-2.28270 0.06424 3.13332
- added joint a_toy_airplane_10_joint: type fixed, parent right_arm_base, child a_toy_airplane_10, origin xyz=0.25991 0.14912 0.95980 rpy=-2.98235 1.44151 -3.00874
- added joint a_toy_airplane_21_joint: type fixed, parent right_arm_base, child a_toy_airplane_21, origin xyz=-0.80537 0.18320 0.26905 rpy=0.89070 -1.80673 2.55451
- added joint a_toy_airplane_22_joint: type fixed, parent right_arm_base, child a_toy_airplane_22, origin xyz=-0.82991 0.36700 0.54016 rpy=0.50942 -2.81968 -0.51512
- added joint banana_1_joint: type fixed, parent right_arm_base, child banana_1, origin xyz=-1.11090 0.39493 0.53727 rpy=0.15938 2.56654 -0.85291
- added joint bleach_cleanser_12_joint: type fixed, parent right_arm_base, child bleach_cleanser_12, origin xyz=0.49049 0.11375 0.18459 rpy=0.72407 1.52342 -2.43087
- added joint bleach_cleanser_29_joint: type fixed, parent right_arm_base, child bleach_cleanser_29, origin xyz=0.76036 0.11881 0.67458 rpy=1.74177 1.40441 -0.01288
- added joint bleach_cleanser_4_joint: type fixed, parent left_arm_base, child bleach_cleanser_4, origin xyz=-0.08968 -0.58731 0.39906 rpy=-0.27300 0.99831 2.76835
- added joint bowl_8_joint: type fixed, parent left_arm_base, child bowl_8, origin xyz=-0.15414 -0.34125 0.85405 rpy=1.59825 -2.28394 -1.47126
- added joint cracker_box_20_joint: type fixed, parent right_arm_base, child cracker_box_20, origin xyz=0.72929 0.44894 0.08773 rpy=-3.01717 1.57447 -2.48045
- added joint cracker_box_5_joint: type fixed, parent right_arm_base, child cracker_box_5, origin xyz=-0.56161 -0.50363 0.91910 rpy=-0.12713 -1.23592 1.88030
- added joint cracker_box_6_joint: type fixed, parent left_arm_base, child cracker_box_6, origin xyz=0.15316 0.56430 0.34842 rpy=2.72787 0.77450 -2.66800
- added joint hammer_16_joint: type fixed, parent left_arm_base, child hammer_16, origin xyz=0.49509 -0.12801 0.13718 rpy=0.66651 -0.50419 -3.02829
- added joint hammer_23_joint: type fixed, parent right_arm_base, child hammer_23, origin xyz=-0.55862 -0.92186 0.58946 rpy=-3.01918 2.89447 -2.39646
- added joint hammer_25_joint: type fixed, parent left_arm_base, child hammer_25, origin xyz=0.05178 -0.32250 0.47753 rpy=1.96073 -2.76466 0.86265
- added joint hammer_3_joint: type fixed, parent right_arm_base, child hammer_3, origin xyz=0.64824 -0.33116 0.42121 rpy=2.08303 -0.91782 2.40552
- added joint mug_26_joint: type fixed, parent left_arm_base, child mug_26, origin xyz=-0.49708 -0.30999 0.04335 rpy=-1.35491 -0.79858 2.73488
- added joint mug_27_joint: type fixed, parent right_arm_base, child mug_27, origin xyz=-0.59216 0.03559 0.06914 rpy=-0.79549 1.35669 -2.26405
- added joint powerdrill_18_joint: type fixed, parent right_arm_base, child powerdrill_18, origin xyz=0.12748 1.15295 0.57592 rpy=-1.56589 0.57326 0.78015
- added joint powerdrill_24_joint: type fixed, parent left_arm_base, child powerdrill_24, origin xyz=0.60987 -0.06337 0.24590 rpy=-3.02187 1.16434 -2.50597
- added joint rubiks_cube_15_joint: type fixed, parent right_arm_base, child rubiks_cube_15, origin xyz=0.03205 -0.13024 0.39989 rpy=0.11489 1.76595 -0.08217
- added joint rubiks_cube_17_joint: type fixed, parent right_arm_base, child rubiks_cube_17, origin xyz=-0.01854 0.99459 0.13216 rpy=-2.06899 -0.29286 -1.68606
- added joint rubiks_cube_19_joint: type fixed, parent left_arm_base, child rubiks_cube_19, origin xyz=-0.47499 0.24952 0.33200 rpy=-3.11128 -2.91854 -0.57349
- added joint rubiks_cube_28_joint: type fixed, parent left_arm_base, child rubiks_cube_28, origin xyz=0.54105 0.51926 0.09200 rpy=-2.63573 2.19956 0.88588
- added joint strawberry_11_joint: type fixed, parent left_arm_base, child strawberry_11, origin xyz=0.32143 -0.13679 0.37842 rpy=0.14509 -3.12943 0.56208
- added joint strawberry_7_joint: type fixed, parent left_arm_base, child strawberry_7, origin xyz=0.86467 -0.56679 0.20161 rpy=1.53802 -2.77240 0.96076
- added joint strawberry_9_joint: type fixed, parent right_arm_base, child strawberry_9, origin xyz=0.51064 0.20361 1.12176 rpy=1.62992 -2.78473 -0.87827
- joint banana_2_joint: origin xyz=0.09189 0.46243 0.24399 rpy=-1.32084 -3.00657 2.12106 -> xyz=0.41082 -0.50321 0.32349 rpy=2.85843 -0.62918 1.49911
- joint mug_13_joint: origin xyz=-0.60808 -0.69298 0.60835 rpy=-2.00569 -2.56604 0.32063 -> xyz=-0.25129 0.65399 0.46320 rpy=0.66071 -2.85400 -1.48320; parent right_arm_base -> left_arm_base
- joint mug_14_joint: origin xyz=0.31101 -0.11514 0.02342 rpy=2.31270 -0.29532 1.59684 -> xyz=-0.28700 -0.99592 0.55608 rpy=-1.72456 1.01052 -1.15418
- joint ur10_base_joint_connection: origin xyz=0.9772262573242188 -0.026124268770217896 0.81 rpy=0.00000 0.00000 1.5708 -> xyz=1.0 0.0 1.0 rpy=0.00000 0.00000 1.5708
- joint ur5_base_joint_connection: origin xyz=-0.4220163822174072 -0.10995670408010483 0.76 rpy=0.00000 0.00000 0.00000 -> xyz=-1.0 0.0 1.0 rpy=0.00000 0.00000 0.00000

File: data/urdfs/dual_arm/dual_arm.urdf (robot description, URDF)
Before this commit: robot dual_arm, 25 links, 24 joints
Links:
- added link left_hand_ee_link, mass 0.0
- added link left_index_fle, mass 0.011300000177428476; collision cylinder length=0.016970543 radius=0.007128496
- added link left_index_sensor, mass 0.017650000000000006; collision cylinder length=0.014262128 radius=0.007128496; collision cylinder length=0.030371139 radius=0.007957384
- added link left_little_fle, mass 0.020700013671416113; collision cylinder length=0.029933618 radius=0.007603541; collision cylinder length=0.030442065 radius=0.007827825
- added link left_middle_fle, mass 0.012100000000000007; collision cylinder length=0.017823514 radius=0.006834489
- added link left_middle_sensor, mass 0.017699999999999994; collision cylinder length=0.011829441 radius=0.006834489; collision cylinder length=0.038238775 radius=0.00812763
- added link left_palm, mass 0.27400616630854535; collision box size=0.062414549 0.056382515 0.028578525; collision box size=0.072641067 0.047533799 0.033261057
- added link left_ring_fle, mass 0.026300044884193397; collision cylinder length=0.029933633 radius=0.00760354; collision cylinder length=0.036828272 radius=0.007827824
- added link left_thumb_fle, mass 0.059200142739743014; collision cylinder length=0.055018354 radius=0.011694114; collision cylinder length=0.059818532 radius=0.012714386
- added link left_thumb_opp, mass 0.01300000026709666; visual mesh filename=meshes/mia_visual/thumb_metacarpus_l.stl scale=0.000999987 0.000999987 0.000999987
- added link left_thumb_sensor, mass 0.000643
- added link right_hand_ee_link, mass 0.0
- added link right_index_fle, mass 0.01113; collision cylinder length=0.016970539 radius=0.007128498
- added link right_index_sensor, mass 0.01765; collision cylinder length=0.014262123 radius=0.007128498; collision cylinder length=0.030371133 radius=0.007957385
- added link right_little_fle, mass 0.0207; collision cylinder length=0.029933602 radius=0.007603541; collision cylinder length=0.030442052 radius=0.007827824
- added link right_middle_fle, mass 0.0121; collision cylinder length=0.01782351 radius=0.006834491
- added link right_middle_sensor, mass 0.0177; collision cylinder length=0.011829435 radius=0.00683449; collision cylinder length=0.038238756 radius=0.008127632
- added link right_palm, mass 0.273999989; collision box size=0.062414549 0.056382477 0.028578509; collision box size=0.072641067 0.047533765 0.033261035
- added link right_ring_fle, mass 0.0263; collision cylinder length=0.029933617 radius=0.00760354; collision cylinder length=0.03682825 radius=0.007827824
- added link right_thumb_fle, mass 0.0592; collision cylinder length=0.055018328 radius=0.011694114; collision cylinder length=0.059818495 radius=0.012714386
- added link right_thumb_opp, mass 0.013; visual mesh filename=meshes/mia_visual/thumb_metacarpus_r.stl scale=0.000999987 0.000999987 0.000999987
- added link right_thumb_sensor, mass 0.000643
Joints:
- added joint left_j_index_fle: type revolute, parent left_palm, child left_index_fle, origin xyz=0.026305504000000004 -0.11021699000000004 -0.021520773000000007 rpy=0.5969194769999983 1.4155536889999998 0.7498065829999984, axis 0 0 -1, limit lower=0.0 upper=1.4 effort=1.75 velocity=3.140000105
- added joint left_j_index_sensor: type fixed, parent left_index_fle, child left_index_sensor, origin xyz=-0.0003992640000000103 -0.02423698099999999 -0.00018396999999999858 rpy=-0.000630706000000008 -0.00020911199999984476 -0.17208260299999997
- added joint left_j_little_fle: type revolute, parent left_palm, child left_little_fle, origin xyz=-0.027859999000000003 -0.107325219 -0.02060511899999999 rpy=1.863250048589795 1.3656738125897925 1.5144063555897949, axis 0 0 -1, limit lower=0.0 upper=1.4 effort=1.75 velocity=3.140000105, mimic joint=left_j_mrl_fle multiplier=1 offset=0
- added joint left_j_middle_sensor: type fixed, parent left_middle_fle, child left_middle_sensor, origin xyz=0.00044401200000001445 -0.02549753199999999 5.810000000003659e-07 rpy=-1.8000000000000002e-08 2.0700000002982222e-07 1.4999999988728386e-08
- added joint left_j_mrl_fle: type revolute, parent left_palm, child left_middle_fle, origin xyz=0.00514942 -0.11355503600000003 -0.024345281999999996 rpy=1.5707941060000015 1.4835299250000018 1.5707939860000009, axis 0 0 -1, limit lower=0.0 upper=1.4 effort=1.75 velocity=3.140000105
- added joint left_j_palm: type fixed, parent ur5_flange, child left_palm, origin xyz=0.0 0.0 0.0 rpy=0.0 0.0 1.57
- added joint left_j_ring_fle: type revolute, parent left_palm, child left_ring_fle, origin xyz=-0.012250358000000001 -0.11202888899999999 -0.02393635699999999 rpy=1.990784438589791 1.460348041589791 1.819812687589792, axis 0 0 -1, limit lower=0.0 upper=1.4 effort=1.75 velocity=3.140000105, mimic joint=left_j_mrl_fle multiplier=1 offset=0
- added joint left_j_thumb_fle: type revolute, parent left_thumb_sensor, child left_thumb_fle, origin xyz=-2.7414000000017258e-05 -0.008989776000000005 -1.0546000000000166e-05 rpy=1.5706005099999993 -1.1325702670000002 -1.5705155129999995, axis 0 0 -1, limit lower=0.0 upper=1.1345 effort=3.5 velocity=1.570000052
- added joint left_j_thumb_opp: type revolute, parent left_palm, child left_thumb_opp, origin xyz=0.013073999000000001 -0.06810817100000002 -0.0019494180000000014 rpy=-1.4371908900000006 0.369162738 -0.31859204200000013, axis 0 0 -1, limit lower=-0.628 upper=0.0 effort=3.5 velocity=4.0
- added joint left_j_thumb_sensor: type fixed, parent left_thumb_opp, child left_thumb_sensor, origin xyz=-5.931000000000686e-06 -0.00899765399999999 2.433000000051644e-06 rpy=-1.9869999999658673e-06 1.49000000115862e-07 1.3900000002698198e-07
- added joint left_palm_to_hand_ee_link: type fixed, parent left_palm, child left_hand_ee_link, origin xyz=0.0 -0.13000000000000003 0.03 rpy=0.65 0.0 0.0
- added joint right_j_index_fle: type revolute, parent right_palm, child right_index_fle, origin xyz=0.026305504 0.11021702 -0.021520771 rpy=-0.596919358 1.415553689 -0.749806523, axis -6e-08 1.7e-08 0.99999994, limit lower=0.0 upper=1.4 effort=1.75 velocity=3.140000105
- added joint right_j_index_sensor: type fixed, parent right_index_fle, child right_index_sensor, origin xyz=-0.000399255 0.024237007 -0.000183955 rpy=0.000630725 -0.000209123 0.172082633
- added joint right_j_little_fle: type revolute, parent right_palm, child right_little_fle, origin xyz=-0.027859999 0.107325219 -0.020605115 rpy=1.278342605 1.775918841 1.627186179, axis -6e-08 1.7e-08 1.0, limit lower=0.0 upper=1.4 effort=1.75 velocity=3.140000105, mimic joint=right_j_mrl_fle multiplier=1 offset=0
- added joint right_j_middle_sensor: type fixed, parent right_middle_fle, child right_middle_sensor, origin xyz=0.000444004 0.025497464 5.81e-07 rpy=1.8e-08 2.07e-07 -3e-08
- added joint right_j_mrl_fle: type revolute, parent right_palm, child right_middle_fle, origin xyz=0.00514942 0.113555029 -0.024345273 rpy=-1.570794106 1.483529925 -1.570793986, axis -6e-08 1.7e-08 0.99999994, limit lower=0.0 upper=1.4 effort=1.75 velocity=3.140000105
- added joint right_j_palm: type fixed, parent ur10_flange, child right_palm, origin xyz=0.0 0.0 0.0 rpy=0.0 0.0 -1.57
- added joint right_j_ring_fle: type revolute, parent right_palm, child right_ring_fle, origin xyz=-0.012250358 0.112028912 -0.023936352 rpy=1.150808096 1.681244493 1.321779966, axis -6e-08 1.7e-08 1.0, limit lower=0.0 upper=1.4 effort=1.75 velocity=3.140000105, mimic joint=right_j_mrl_fle multiplier=1 offset=0
- added joint right_j_thumb_fle: type revolute, parent right_thumb_sensor, child right_thumb_fle, origin xyz=-2.7426e-05 -1.0543e-05 -0.008989788 rpy=-1.570910335 0.438224047 1.570665002, axis -6e-08 1.7e-08 1.0, limit lower=0.0 upper=1.1345 effort=3.5 velocity=1.570000052
- added joint right_j_thumb_opp: type revolute, parent right_palm, child right_thumb_opp, origin xyz=0.013073999 0.068108179 -0.001949422 rpy=1.43719089 0.369162768 0.318591952, axis -6e-08 1.7e-08 1.0, limit lower=-0.628 upper=0.0 effort=3.5 velocity=4.0
- added joint right_j_thumb_sensor: type fixed, parent right_thumb_opp, child right_thumb_sensor, origin xyz=-5.942e-06 0.008997655 2.453e-06 rpy=1.570796371 1.01e-07 -1.19e-07
- added joint right_palm_to_hand_ee_link: type fixed, parent right_palm, child right_hand_ee_link, origin xyz=0 0.13 0.03 rpy=-0.65 0 0
- joint ur10_base_joint: origin xyz=0.9772262573242188 -0.026124268770217896 0.8100000011920929 rpy=0.00000 0.00000 1.5708 -> xyz=1.0 0.0 1.0 rpy=0.00000 0.00000 1.5708
- joint ur5_base_joint: origin xyz=-0.4220163822174072 -0.10995670408010483 0.7599999952316284 rpy=0.00000 0.00000 0.00000 -> xyz=-1.0 0.0 1.0 rpy=0.00000 0.00000 0.00000
